File: pro-micro-receiver.kicad_pcb (KiCad board)
At the start: 4 copper layers, 53.6 x 19.5 mm, 56 parts, among them J1 USB_A_PLUG, J2 Conn_01x04, SW1 SW_Push, U1 TLV740P, U2 ATmega32U4-M, U3 YJ-14015, Y1 16MHz

Commit message: Adding labels to +3V3 and GND testpoints
Parts:
- added kibuzzard-63BC8113: G***, kibuzzard-63BC8113, F.Cu at (90.1, 65.4)
- R1: value R -> 10k
- R10, R11, R12: value R -> 1k5
Other:
- board text added: "GND"
Changed lines of the file:
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@@
     )
+  )
+  (footprint "kibuzzard-63BC8113" (layer "F.Cu")
+    (at 90.07 65.4)
+    (descr "Converted using: scripting")
+    (tags "svg2mod")
+    (attr board_only exclude_from_pos_files exclude_from_bom)
+    (fp_text reference "kibuzzard-63BC8113" (at 0 -0.968089) (layer "F.SilkS") hide
+      (effects (font (size 0.000254 0.000254) (thickness 0.000003)))
+    )
+    (fp_text value "G***" (at 0 0.968089) (layer "F.SilkS") hide
+      (effects (font (size 0.000254 0.000254) (thickness 0.000003)))
+    )
+    (fp_poly (pts
+        (xy -2.275284 -0.967581)
+        (xy -2.275284 -0.007144)
+        (xy -1.901428 -0.007144)
+        (xy -1.901428 -0.421481)
+        (xy -1.649016 -0.421481)
+        (xy -1.649016 -0.007144)
+        (xy -1.275159 -0.007144)
+        (xy -1.275159 0.233363)
+        (xy -1.649016 0.233363)
+        (xy -1.082278 0.688181)
+        (xy -1.025128 0.442913)
+        (xy -0.883444 0.492919)
+        (xy -0.787896 0.512564)
+        (xy -0.675084 0.519113)
+        (xy -0.54739 0.503039)
+        (xy -0.464344 0.454819)
+        (xy -0.403622 0.295275)
+        (xy -0.426839 0.196155)
+        (xy -0.496491 0.132159)
+        (xy -0.601861 0.097334)
+        (xy -0.732234 0.085725)
+        (xy -0.822722 0.085725)
+        (xy -0.822722 -0.157163)
+        (xy -0.713184 -0.157163)
+        (xy -0.622697 -0.166688)
+        (xy -0.541734 -0.197644)
+        (xy -0.483394 -0.254794)
+        (xy -0.460772 -0.345281)
+        (xy -0.509588 -0.472678)
+        (xy -0.644128 -0.519113)
+        (xy -0.809625 -0.491728)
+        (xy -0.951309 -0.423863)
+        (xy -1.056084 -0.638175)
+        (xy -0.885825 -0.725091)
+        (xy -0.773013 -0.75813)
+        (xy -0.646509 -0.769144)
+        (xy -0.530721 -0.761405)
+        (xy -0.431006 -0.738188)
+        (xy -0.279797 -0.651272)
+        (xy -0.191691 -0.519113)
+        (xy -0.163116 -0.354806)
+        (xy -0.213122 -0.185738)
+        (xy -0.346472 -0.061913)
+        (xy -0.244971 -0.002977)
+        (xy -0.169069 0.078581)
+        (xy -0.121741 0.18038)
+        (xy -0.105966 0.300038)
+        (xy -0.139303 0.488156)
+        (xy 0.453628 0.738188)
+        (xy 0.394692 0.563166)
+        (xy 0.332184 0.366713)
+        (xy 0.290116 0.228732)
+        (xy 0.249634 0.091017)
+        (xy 0.210741 -0.046434)
+        (xy 0.173964 -0.18124)
+        (xy 0.139832 -0.311018)
+        (xy 0.108347 -0.435769)
+        (xy 0.069056 -0.602456)
+        (xy 0.041672 -0.735806)
+        (xy 0.351234 -0.735806)
+        (xy 0.369094 -0.612279)
+        (xy 0.394097 -0.470297)
+        (xy 0.42416 -0.316706)
+        (xy 0.4572 -0.158353)
+        (xy 0.492919 0.001191)
+        (xy 0.531019 0.158353)
+        (xy 0.570012 0.306288)
+        (xy 0.608409 0.43815)
+        (xy 0.646509 0.308074)
+        (xy 0.684609 0.160734)
+        (xy 0.721519 0.003572)
+        (xy 0.756047 -0.155972)
+        (xy 0.788194 -0.314623)
+        (xy 0.817959 -0.469106)
+        (xy 0.844153 -0.611981)
+        (xy 0.865584 -0.735806)
+        (xy 1.172766 -0.735806)
+        (xy 1.140916 -0.584597)
+        (xy 1.102519 -0.416719)
+        (xy 1.05787 -0.236041)
+        (xy 1.007269 -0.046434)
+        (xy 0.970359 0.083741)
+        (xy 0.931069 0.215503)
+        (xy 0.889397 0.348853)
+        (xy 0.846005 0.481542)
+        (xy 0.801555 0.61132)
+        (xy 1.372791 0.714375)
+        (xy 1.298972 0.688181)
+        (xy 1.356122 0.442913)
+        (xy 1.497806 0.492919)
+        (xy 1.593354 0.512564)
+        (xy 1.706166 0.519113)
+        (xy 1.83386 0.503039)
+        (xy 1.916906 0.454819)
+        (xy 1.977628 0.295275)
+        (xy 1.954411 0.196155)
+        (xy 1.884759 0.132159)
+        (xy 1.779389 0.097334)
+        (xy 1.649016 0.085725)
+        (xy 1.558528 0.085725)
+        (xy 1.558528 -0.157163)
+        (xy 1.668066 -0.157163)
+        (xy 1.758553 -0.166688)
+        (xy 1.839516 -0.197644)
+        (xy 1.897856 -0.254794)
+        (xy 1.920478 -0.345281)
+        (xy 1.871663 -0.472678)
+        (xy 1.737122 -0.519113)
+        (xy 1.571625 -0.491728)
+        (xy 1.429941 -0.423863)
+        (xy 1.325166 -0.638175)
+        (xy 1.495425 -0.725091)
+        (xy 1.608237 -0.75813)
+        (xy 1.734741 -0.769144)
+        (xy 1.850529 -0.761405)
+        (xy 1.950244 -0.738188)
+        (xy 2.101453 -0.651272)
+        (xy 2.189559 -0.519113)
+        (xy 2.218134 -0.354806)
+        (xy 2.168128 -0.185738)
+        (xy 2.034778 -0.061913)
+        (xy 2.136279 -0.002977)
+        (xy 2.212181 0.078581)
+        (xy 2.259509 0.18038)
+        (xy 2.275284 0.300038)
+        (xy 2.241947 0.488156)
+        (xy 2.139553 0.636984)
+        (xy 2.060972 0.692944)
+        (xy 1.963341 0.734616)
+        (xy 1.846064 0.760512)
+        (xy 1.708547 0.769144)
+        (xy 1.593056 0.760809)
+        (xy 1.476375 0.740569)
+        (xy 1.372791 0.714375)
+        (xy 0.801555 0.61132)
+        (xy 0.756047 0.738188)
+        (xy 0.453628 0.738188)
+        (xy -0.139303 0.488156)
+        (xy -0.241697 0.636984)
+        (xy -0.320278 0.692944)
+        (xy -0.417909 0.734616)
+        (xy -0.535186 0.760512)
+        (xy -0.672703 0.769144)
+        (xy -0.788194 0.760809)
+        (xy -0.904875 0.740569)
+        (xy -1.008459 0.714375)
+        (xy -1.082278 0.688181)
+        (xy -1.649016 0.233363)
+        (xy -1.649016 0.6477)
+        (xy -1.901428 0.6477)
+        (xy -1.901428 0.233363)
+        (xy -2.275284 0.233363)
+        (xy -2.275284 -0.007144)
+        (xy -2.275284 -0.967581)
+        (xy -2.275483 -0.967581)
+        (xy -2.464249 -0.948989)
+        (xy -2.64576 -0.893929)
+        (xy -2.813042 -0.804514)
+        (xy -2.959666 -0.684183)
+        (xy -3.079997 -0.537559)
+        (xy -3.169411 -0.370277)
+        (xy -3.224472 -0.188766)
+        (xy -3.243064 0)
+        (xy -3.224472 0.188766)
+        (xy -3.169411 0.370277)
+        (xy -3.079997 0.537559)
+        (xy -2.959666 0.684183)
+        (xy -2.813042 0.804514)
+        (xy -2.64576 0.893929)
+        (xy -2.464249 0.948989)
+        (xy -2.275483 0.967581)
+        (xy -2.275284 0.967581)
+        (xy 2.275284 0.967581)
+        (xy 2.275483 0.967581)
+        (xy 2.464249 0.948989)
+        (xy 2.64576 0.893929)
+        (xy 2.813042 0.804514)
+        (xy 2.959666 0.684183)
+        (xy 3.079997 0.537559)
+        (xy 3.169411 0.370277)
+        (xy 3.224472 0.188766)
+        (xy 3.243064 0)
+        (xy 3.224472 -0.188766)
+        (xy 3.169411 -0.370277)
+        (xy 3.079997 -0.537559)
+        (xy 2.959666 -0.684183)
+        (xy 2.813042 -0.804514)
+        (xy 2.64576 -0.893929)
+        (xy 2.464249 -0.948989)
+        (xy 2.275483 -0.967581)
+        (xy 2.275284 -0.967581)
+        (xy -2.275284 -0.967581)
+      ) (layer "F.SilkS") (width 0) (fill solid))
   )
   (footprint "Diode_SMD_AKL:D_0603_1608Metric_Pad1.05x0.95mm" (layer "F.Cu")
@@
       (effects (font (size 1 1) (thickness 0.15)))
     )
-    (fp_text value "R" (at 0 1.43) (layer "F.Fab") hide
+    (fp_text value "1k5" (at 0 1.43) (layer "F.Fab") hide
       (effects (font (size 1 1) (thickness 0.15)))
     )
@@
       (effects (font (size 1 1) (thickness 0.15)))
     )
-    (fp_text value "R" (at 0 1.43) (layer "F.Fab") hide
+    (fp_text value "10k" (at 0 1.43) (layer "F.Fab") hide
       (effects (font (size 1 1) (thickness 0.15)))
     )
@@
       (effects (font (size 1 1) (thickness 0.15)))
     )
-    (fp_text value "R" (at 0 1.43) (layer "F.Fab") hide
+    (fp_text value "1k5" (at 0 1.43) (layer "F.Fab") hide
       (effects (font (size 1 1) (thickness 0.15)))
     )
@@
       (effects (font (size 1 1) (thickness 0.15)))
     )
-    (fp_text value "R" (at 0 1.43) (layer "F.Fab") hide
+    (fp_text value "1k5" (at 0 1.43) (layer "F.Fab") hide
       (effects (font (size 1 1) (thickness 0.15)))
     )
@@
   (gr_line (start 99.54 81.21) (end 106.4 81.21) (layer "User.1") (width 0.15))
   (gr_line (start 99.54 66.39) (end 106.38 66.39) (layer "User.1") (width 0.15))
+  (gr_text "GND" (at 81.11 80.69) (layer "F.SilkS")
+    (effects (font (size 1 1) (thickness 0.15)))
+  )
   (dimension (type orthogonal) (layer "User.1")
     (pts (xy 72.8375 67.72) (xy 117 68.54))
@@
       (effects (font (size 1 1) (thickness 0.15)))
     )
+    (format (units 3) (units_format 1) (precision 4))
+    (style (thickness 0.15) (arrow_length 1.27) (text_position_mode 0) (extension_height 0.58642) (extension_offset 0.5) keep_text_aligned)
+  )
+  (dimension (type orthogonal) (layer "User.1")
+    (pts (xy 113 64) (xy 113 83.5))
+    (height 9.68)
+    (orientation 1)
+    (gr_text "19,5000 mm" (at 121.53 73.75 90) (layer "User.1")
+      (effects (font (size 1 1) (thickness 0.15)))
+    )
